File: pcb/vim60/vim60.kicad_pcb (KiCad board)
At the start: 2 copper layers, 285.4 x 94.9 mm, 315 parts, among them IC1 ATMEGA32U4, J1 USBMINI_B05, Q1 NPN, X1 ASX4

Commit message: making bom
Parts:
- removed the HOLE at (349.7, 159.5)
- removed the HOLE at (67.6, 159.5)
- added REF**: geek, logos:geek, F.Cu at (80.6, 189.8)
- DB63: footprint mx1a:MX1A-led -> mx1a:caps_led
- moved C8 121.0 mm to (182.8, 108.2), turned to 90 degrees
- moved R63 105.8 mm to (84.4, 114.9), turned to 90 degrees
- moved C7 102.5 mm to (163.7, 108.2), turned to 90 degrees
- moved R64 101.6 mm to (86.9, 114.9), turned to 90 degrees
- moved C6 84.2 mm to (144.7, 108.2), turned to 90 degrees
- moved C5 66.6 mm to (125.6, 108.2), turned to 90 degrees
- moved C4 50.1 mm to (106.6, 108.2), turned to 90 degrees
- moved C2 30.8 mm to (150.7, 189.0), turned to 270 degrees
- moved C1 29.2 mm to (154.2, 189.1), turned to 90 degrees
- moved R65 24.6 mm to (180.6, 184.7), turned to 0 degrees
- moved X1 22.9 mm to (158.3, 189.0), turned to 90 degrees
- moved C9 20.9 mm to (163.9, 174.3), turned to 0 degrees
- moved C28 20.8 mm to (123.7, 177.1), turned to 270 degrees
- moved C3 19.3 mm to (182.2, 193.1), turned to 90 degrees
- moved R68 18.7 mm to (157.3, 193.6), turned to 90 degrees
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Connections:
- IC1 pad 1: /col13 -> /row03
- IC1 pad 10: /row05 -> /row01
- IC1 pad 11: /row04 -> /row02
- IC1 pad 18: /col12 -> /col01
- IC1 pad 19: /col11 -> /col02
- IC1 pad 20: /col10 -> /col04
- IC1 pad 21: /col09 -> /col03
- IC1 pad 22: /col07 -> /col05
- IC1 pad 25: /col08 -> /col06
- IC1 pad 26: /col06 -> /col07
- IC1 pad 27: /col05 -> /col08
- IC1 pad 28: /row03 -> /col09
- IC1 pad 29: /row02 -> /rgb
- IC1 pad 30: /rgb -> /col10
- IC1 pad 31: /col04 -> /col11
- IC1 pad 32: /col03 -> /col12
- IC1 pad 36: /col14 -> /col13
- IC1 pad 37: /row01 -> /col14
- IC1 pad 8: /col02 -> /row04
- IC1 pad 9: /col01 -> /row05
Routing:
- net VCC: track 1374.3 -> 1675.6 mm
- net /col15: track 72.1 -> 282.2 mm, vias 0 -> 4
- net /col13: track 64.4 -> 264.5 mm
- net /col14: track 57.1 -> 255.7 mm, vias 2 -> 6
- net Net-(IC1-Pad4): track 0.00 -> 193.0 mm, vias 0 -> 2
- net Net-(IC1-Pad3): track 0.00 -> 192.8 mm, vias 0 -> 2
- net /col12: track 74.1 -> 251.2 mm, vias 4 -> 6
- net /col10: track 50.6 -> 190.8 mm, vias 2 -> 4
- net /col03: track 74.7 -> 189.9 mm, vias 4 -> 7
- net /col02: track 75.4 -> 190.4 mm, vias 4 -> 7
- net /col01: track 70.1 -> 182.7 mm, vias 0 -> 4
- net Net-(IC1-Pad13): track 0.00 -> 110.2 mm, vias 0 -> 2
- net /col04: track 89.2 -> 187.2 mm, vias 4 -> 7
- net /col08: track 79.0 -> 174.1 mm
- net /col11: track 100.2 -> 190.4 mm, vias 4 -> 6
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- added copper zone on B.Cu, net GND
- added copper zone on F.Cu, net GND
Other:
- board size 285.4 x 94.9 mm -> 285 x 94.6 mm
