File: pcb/vim60/vim60.sch (KiCad schematic (older format))
At the start: 11 parts, among them IC1 ATMEGA32U4, J1 USBMINI_B05, X1 ASX4

Commit message: 200517
Parts:
- added C4: 1u, 0805:0805C, symbol device:C
- added C5, C6, C7, C8: 100n, 0805:0805C, symbol device:C
- C1, C2, C3: footprint (none) -> 0805:0805C
- IC1: footprint TQFP44 -> tqfp:TQFP44
- J1: footprint (none) -> usb:67503
- R63: renamed from R1; footprint (none) -> 0805:0805R
- R64: renamed from R2; footprint (none) -> 0805:0805R
- R65: renamed from R3; footprint (none) -> 0805:0805R
- R66: renamed from R5; footprint (none) -> 0805:0805R
- S0: footprint switch-tact-DTSM-6 -> dtsm:KSEM31GLFS
- X1: footprint (none) -> ndk:4-SMD
Connections:
- net GND: now also C4.2, C5.2, C6.2, C7.2, C8.2
- net VCC: now also C4.1, C5.1, C6.1, C7.1, C8.1
- net col13: now reaches IC1.1 ((INT6/AIN0)PE6)
- net row05: now reaches IC1.10 ((PDI/PCINT2/MOSI)PB2)
- net row04: now reaches IC1.11 ((PDO/PCINT3/MISO)PB3)
- net bl: now reaches IC1.12 ((PCINT7/OC0A/OC1C/~RTS~)PB7)
- net col12: now reaches IC1.18 ((OC0B/SCL/INT0)PD0)
- net col11: now reaches IC1.19 ((SDA/INT1)PD1)
- net col10: now reaches IC1.20 ((RXD1/INT2)PD2)
- net col09: now reaches IC1.21 ((TXD1/INT3)PD3)
- net col07: now reaches IC1.22 ((XCK1/~CTS~)PD5)
- net col08: now reaches IC1.25 ((ICP1/ADC8)PD4)
- net col06: now reaches IC1.26 ((T1/~OC4D~/ADC9)PD6)
- net col05: now reaches IC1.27 ((T0/OC4D/ADC10)PD7)
- net row03: now reaches IC1.28 ((PCINT4/ADC11)PB4)
- net row02: now reaches IC1.29 ((PCINT5/OC1A/~OC4B~/ADC12)PB5)
- net rgb: now reaches IC1.30 ((PCINT6/OC1B/OC4B/ADC13)PB6)
- net col04: now reaches IC1.31 ((OC3A/~OC4A~)PC6)
- net col03: now reaches IC1.32 ((ICP3/CLK0/OC4A)PC7)
- net col14: now reaches IC1.36 ((ADC7/TDI)PF7)
- net row01: now reaches IC1.37 ((ADC6/TDO)PF6)
- net col15: now reaches IC1.40 ((ADC1)PF1)
- net CAPS_LED: now reaches IC1.41 ((ADC0)PF0)
- net col02: now reaches IC1.8 ((SS/PCINT0)PB0)
- net col01: now reaches IC1.9 ((PCINT1/SCLK)PB1)
- no-connect marks 4 -> 6
Other:
- moved on the sheet: R65

Commit message: making bom
Connections:
- net col01: now also IC1.18 ((OC0B/SCL/INT0)PD0); no longer IC1.9 ((PCINT1/SCLK)PB1)
- net col02: now also IC1.19 ((SDA/INT1)PD1); no longer IC1.8 ((SS/PCINT0)PB0)
- net col03: now also IC1.21 ((TXD1/INT3)PD3); no longer IC1.32 ((ICP3/CLK0/OC4A)PC7)
- net col04: now also IC1.20 ((RXD1/INT2)PD2); no longer IC1.31 ((OC3A/~OC4A~)PC6)
- net col05: now also IC1.22 ((XCK1/~CTS~)PD5); no longer IC1.27 ((T0/OC4D/ADC10)PD7)
- net col06: now also IC1.25 ((ICP1/ADC8)PD4); no longer IC1.26 ((T1/~OC4D~/ADC9)PD6)
- net col07: now also IC1.26 ((T1/~OC4D~/ADC9)PD6); no longer IC1.22 ((XCK1/~CTS~)PD5)
- net col08: now also IC1.27 ((T0/OC4D/ADC10)PD7); no longer IC1.25 ((ICP1/ADC8)PD4)
- net col09: now also IC1.28 ((PCINT4/ADC11)PB4); no longer IC1.21 ((TXD1/INT3)PD3)
- net col10: now also IC1.30 ((PCINT6/OC1B/OC4B/ADC13)PB6); no longer IC1.20 ((RXD1/INT2)PD2)
- net col11: now also IC1.31 ((OC3A/~OC4A~)PC6); no longer IC1.19 ((SDA/INT1)PD1)
- net col12: now also IC1.32 ((ICP3/CLK0/OC4A)PC7); no longer IC1.18 ((OC0B/SCL/INT0)PD0)
- net col13: now also IC1.36 ((ADC7/TDI)PF7); no longer IC1.1 ((INT6/AIN0)PE6)
- net col14: now also IC1.37 ((ADC6/TDO)PF6); no longer IC1.36 ((ADC7/TDI)PF7)
- net rgb: now also IC1.29 ((PCINT5/OC1A/~OC4B~/ADC12)PB5); no longer IC1.30 ((PCINT6/OC1B/OC4B/ADC13)PB6)
- net row01: now also IC1.10 ((PDI/PCINT2/MOSI)PB2); no longer IC1.37 ((ADC6/TDO)PF6)
- net row02: now also IC1.11 ((PDO/PCINT3/MISO)PB3); no longer IC1.29 ((PCINT5/OC1A/~OC4B~/ADC12)PB5)
- net row03: now also IC1.1 ((INT6/AIN0)PE6); no longer IC1.28 ((PCINT4/ADC11)PB4)
- net row04: now also IC1.8 ((SS/PCINT0)PB0); no longer IC1.11 ((PDO/PCINT3/MISO)PB3)
- net row05: now also IC1.9 ((PCINT1/SCLK)PB1); no longer IC1.10 ((PDI/PCINT2/MOSI)PB2)
Changed lines of the file:
@@
 Wire Wire Line
 	5250 3250 5550 3250
-Wire Wire Line
-	5250 3450 5700 3450
+Text Label 5350 3750 0    50   ~ 0
+row01
+Wire Wire Line
+	5250 3550 5700 3550
+Entry Wire Line
+	5700 3550 5800 3650
+Wire Wire Line
+	5250 3650 5700 3650
+Entry Wire Line
+	5700 3650 5800 3750
+Wire Wire Line
+	5250 3750 5700 3750
+Entry Wire Line
+	5700 3750 5800 3850
+Wire Wire Line
+	5250 3850 5700 3850
+Entry Wire Line
+	5700 3850 5800 3950
+Wire Wire Line
+	5250 3950 5700 3950
+Entry Wire Line
+	5700 3950 5800 4050
+Wire Wire Line
+	5250 4150 5700 4150
+Entry Wire Line
+	5700 4150 5800 4250
+Wire Wire Line
+	5250 4250 5700 4250
+Entry Wire Line
+	5700 4250 5800 4350
+Wire Wire Line
+	5250 4450 5700 4450
+Entry Wire Line
+	5700 4450 5800 4550
+Text Label 5350 3650 0    50   ~ 0
+row02
+Text Label 5350 5450 0    50   ~ 0
+row03
+Text Label 5350 3950 0    50   ~ 0
+row04
+Text Label 5350 3850 0    50   ~ 0
+row05
+Text Label 5350 5150 0    50   ~ 0
+col01
+Text Label 5350 5050 0    50   ~ 0
+col02
+Text Label 5350 4850 0    50   ~ 0
+col03
+Text Label 5350 4950 0    50   ~ 0
+col04
+Text Label 5350 4650 0    50   ~ 0
+col05
+Wire Wire Line
+	5250 4550 5700 4550
+Entry Wire Line
+	5700 4550 5800 4650
+Wire Wire Line
+	5250 4650 5700 4650
+Entry Wire Line
+	5700 4650 5800 4750
+Wire Wire Line
+	5250 4750 5700 4750
+Entry Wire Line
+	5700 4750 5800 4850
+Wire Wire Line
+	5250 4850 5700 4850
+Entry Wire Line
+	5700 4850 5800 4950
+Wire Wire Line
+	5250 4950 5700 4950
+Entry Wire Line
+	5700 4950 5800 5050
+Wire Wire Line
+	5250 5050 5700 5050
+Entry Wire Line
+	5700 5050 5800 5150
+Wire Wire Line
+	5250 5150 5700 5150
+Entry Wire Line
+	5700 5150 5800 5250
+Wire Wire Line
+	5250 5450 5700 5450
+Entry Wire Line
+	5700 5450 5800 5550
+Text Label 5350 4750 0    50   ~ 0
+col06
+Text Label 5350 4550 0    50   ~ 0
+col07
+Text Label 5350 4450 0    50   ~ 0
+col08
+Text Label 5350 3550 0    50   ~ 0
+col09
+Text Label 5350 3350 0    50   ~ 0
+col10
+Text Label 5350 4250 0    50   ~ 0
+col11
+Text Label 5350 4150 0    50   ~ 0
+col12
+Text Label 5350 5650 0    50   ~ 0
+col13
+Wire Wire Line
+	5250 5650 5700 5650
+Entry Wire Line
+	5700 5650 5800 5750
 Text Label 5350 5750 0    50   ~ 0
-row01
-Entry Wire Line
-	5700 3450 5800 3550
-Wire Wire Line
-	5250 3550 5700 3550
-Entry Wire Line
-	5700 3550 5800 3650
-Wire Wire Line
-	5250 3650 5700 3650
-Entry Wire Line
-	5700 3650 5800 3750
-Wire Wire Line
-	5250 3750 5700 3750
-Entry Wire Line
-	5700 3750 5800 3850
-Wire Wire Line
-	5250 3850 5700 3850
-Entry Wire Line
-	5700 3850 5800 3950
-Wire Wire Line
-	5250 3950 5700 3950
-Entry Wire Line
-	5700 3950 5800 4050
-Wire Wire Line
-	5250 4150 5700 4150
-Entry Wire Line
-	5700 4150 5800 4250
-Wire Wire Line
-	5250 4250 5700 4250
-Entry Wire Line
-	5700 4250 5800 4350
-Wire Wire Line
-	5250 4450 5700 4450
-Entry Wire Line
-	5700 4450 5800 4550
-Text Label 5350 3450 0    50   ~ 0
-row02
-Text Label 5350 3550 0    50   ~ 0
-row03
-Text Label 5350 3650 0    50   ~ 0
-row04
-Text Label 5350 3750 0    50   ~ 0
-row05
-Text Label 5350 3850 0    50   ~ 0
-col01
-Text Label 5350 3950 0    50   ~ 0
-col02
-Text Label 5350 4150 0    50   ~ 0
-col03
-Text Label 5350 4250 0    50   ~ 0
-col04
-Text Label 5350 4450 0    50   ~ 0
-col05
-Wire Wire Line
-	5250 4550 5700 4550
-Entry Wire Line
-	5700 4550 5800 4650
-Wire Wire Line
-	5250 4650 5700 4650
-Entry Wire Line
-	5700 4650 5800 4750
-Wire Wire Line
-	5250 4750 5700 4750
-Entry Wire Line
-	5700 4750 5800 4850
-Wire Wire Line
-	5250 4850 5700 4850
-Entry Wire Line
-	5700 4850 5800 4950
-Wire Wire Line
-	5250 4950 5700 4950
-Entry Wire Line
-	5700 4950 5800 5050
-Wire Wire Line
-	5250 5050 5700 5050
-Entry Wire Line
-	5700 5050 5800 5150
-Wire Wire Line
-	5250 5150 5700 5150
-Entry Wire Line
-	5700 5150 5800 5250
-Wire Wire Line
-	5250 5450 5700 5450
-Entry Wire Line
-	5700 5450 5800 5550
-Text Label 5350 4550 0    50   ~ 0
-col06
-Text Label 5350 4650 0    50   ~ 0
-col07
-Text Label 5350 4750 0    50   ~ 0
-col08
-Text Label 5350 4850 0    50   ~ 0
-col09
-Text Label 5350 4950 0    50   ~ 0
-col10
-Text Label 5350 5050 0    50   ~ 0
-col11
-Text Label 5350 5150 0    50   ~ 0
-col12
-Text Label 5350 5450 0    50   ~ 0
-col13
-Wire Wire Line
-	5250 5650 5700 5650
-Entry Wire Line
-	5700 5650 5800 5750
-Text Label 5350 5650 0    50   ~ 0
 col14
 Wire Wire Line
@@
 Entry Wire Line
 	5700 6050 5800 6150
-Text Label 5250 6050 0    50   ~ 0
+Text Label 5350 6050 0    50   ~ 0
 col15
 Entry Wire Line
@@
 Wire Wire Line
 	5250 3350 5700 3350
-Wire Wire Line
-	5700 3350 5700 2650
-Wire Wire Line
-	5700 2650 6900 2650
-Text Label 5350 3350 0    50   ~ 0
+Text Label 5350 3450 0    50   ~ 0
 rgb
+Entry Wire Line
+	5700 3350 5800 3450
+Wire Wire Line
+	5250 3450 5650 3450
+Wire Wire Line
+	5650 3450 5650 2650
+Wire Wire Line
+	5650 2650 6900 2650
 Wire Bus Line
 	6300 3100 6300 6450
