File: pcb/vim60/vim60_matrix.sch (KiCad schematic (older format))
At the start: 125 parts

Commit message: 200517
Parts:
- added R67: 300, 0805:0805R, symbol device:R
- D1: renamed from D01; footprint (none) -> 0805:0805D
- D10, D11, D12, D13, D14, D15, D16, D17, D18, D19, D20, D21, D22, D23, D24, D25, D26, D27, D28, D29, D30, D31, D32, D33, D34, D35, D36, D37, D38, D39, D40, D41, D42, D43, D44, D45, D46, D47, D48, D49, D50, D51, D52, D53, D54, D55, D56, D57, D58, D59, D6, D60, D61, D62, D7, D8, D9: renamed from D?; footprint (none) -> 0805:0805D
- D2: renamed from D02; footprint (none) -> 0805:0805D
- D3: renamed from D03; footprint (none) -> 0805:0805D
- D4: renamed from D04; footprint (none) -> 0805:0805D
- D5: renamed from D05; footprint (none) -> 0805:0805D
- DB63: renamed from D?; footprint (none) -> mx1a:MX1A-led
- S1: renamed from S01; footprint (none) -> mx1a:MX1A
- S10, S11, S17, S18, S19, S20, S21, S22, S23, S24, S25, S26, S27, S28, S29, S30, S31, S32, S33, S34, S35, S36, S37, S38, S39, S40, S41, S42, S43, S44, S45, S46, S47, S48, S49, S50, S51, S52, S53, S54, S55, S56, S57, S58, S59, S60, S61, S62: footprint (none) -> mx1a:MX1A
- S12: renamed from S13; footprint (none) -> mx1a:MX1A
- S13: renamed from S14; footprint (none) -> mx1a:MX1A
- S14: renamed from S15; footprint (none) -> mx1a:MX1A
- S15: renamed from S16; footprint (none) -> mx1a:MX1A
- S16: renamed from S12; footprint (none) -> mx1a:MX1A
- S2: renamed from S02; footprint (none) -> mx1a:MX1A
- S3: renamed from S03; footprint (none) -> mx1a:MX1A
- S4: renamed from S04; footprint (none) -> mx1a:MX1A
- S5: renamed from S05; footprint (none) -> mx1a:MX1A
- S6: renamed from S06; footprint (none) -> mx1a:MX1A
- S7: renamed from S07; footprint (none) -> mx1a:MX1A
- S8: renamed from S08; footprint (none) -> mx1a:MX1A
- S9: renamed from S09; footprint (none) -> mx1a:MX1A
Connections:
- wire segments 332 -> 333
Other:
- moved on the sheet: DB63

Commit message: making bom
Parts:
- DB63: footprint mx1a:MX1A-led -> mx1a:caps_led
Changed lines of the file:
@@
 F 0 "DB63" V 14354 2378 50  0000 L CNN
 F 1 "LED" V 14445 2378 50  0000 L CNN
-F 2 "mx1a:MX1A-led" H 14400 2300 50  0001 C CNN
+F 2 "mx1a:caps_led" H 14400 2300 50  0001 C CNN
 F 3 "" H 14400 2300 50  0001 C CNN
 	1    14400 2300

Commit message: finished
Parts:
- R67: value 300 -> 100
Changed lines of the file:
@@
 P 14400 1750
 F 0 "R67" H 14471 1796 50  0000 L CNN
-F 1 "300" H 14471 1705 50  0000 L CNN
+F 1 "100" H 14471 1705 50  0000 L CNN
 F 2 "0805:0805R" H 14400 1750 50  0001 C CNN
 F 3 "" H 14400 1750 50  0001 C CNN
